File: KEYPAD_BREAKOUT/KEYPAD_BREAKOUT.kicad_sch (KiCad schematic)
At the start: 21 parts, among them J1 Conn_01x14, SW0 SW_RGB, SW1 SW_RGB, SW2 SW_RGB, SW3 SW_RGB, SW4 SW_RGB, SW5 SW_RGB, SW6 SW_RGB, SW7 SW_RGB, SW8 SW_RGB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

Commit message: [KEYPAD_BREAKOUT] Version 1 release, multiple fixes
Signed-off-by: Adam BZH <424778940z@users.noreply.github.com>
Parts:
- added J1: Conn_01x14, Connector_PinSocket_2.00mm:PinSocket_2x07_P2.00mm_Vertical_SMD, symbol Connector_Generic:Conn_01x14
- renumbered J1 to J0
Connections:
- net DIN: now also J1.3 (Pin_3)
- net DOUT: now also J1.4 (Pin_4)
- net GND: now also J1.2 (Pin_2)
- net SW0: now also J1.5 (Pin_5)
- net SW1: now also J1.6 (Pin_6)
- net SW2: now also J1.7 (Pin_7)
- net SW3: now also J1.8 (Pin_8)
- net SW4: now also J1.9 (Pin_9)
- net SW5: now also J1.10 (Pin_10)
- net SW6: now also J1.11 (Pin_11)
- net SW7: now also J1.12 (Pin_12)
- net SW8: now also J1.13 (Pin_13)
- net SW9: now also J1.14 (Pin_14)
- net VCC: now also J1.1 (Pin_1)
Other:
- moved on the sheet: JP0, JP1, JP2, JP3, JP4, JP5, JP6, JP7, JP8, JP9, SW0, SW1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
